File: ECAD/Control Board.kicad_pcb (KiCad board)
At the start: 2 copper layers, 184.2 x 57.8 mm, 77 parts, among them J3 Thermocouple, J4 SD_Card, J5 PWR/Heat, J6 FAN, J7 UPDI, Q1 IPD50N06S4L08, Q2 IPD50N06S4L08, SW1 Reflow, SW2 Stop, SW3 Set temp mode, U1 ATtiny1614-SS, U2 LD1086DT33, U3 AD8497, U4 HT16K33, U5 LM2575HVS-ADJ

Commit message: Lay out switching regulator
Also reshuffling the SD card and power port placements
Parts:
- J4: moved to F.Cu
- moved J6 134.1 mm to (184.8, 109.2), turned to 90 degrees
- moved D5 132.8 mm to (188.6, 105.4), turned to 180 degrees
- moved R33 124.0 mm to (191.1, 95.2), turned to 270 degrees
- moved Q2 121.0 mm to (184.8, 97.8), turned to 270 degrees
- moved R32 120.4 mm to (196.2, 83.2), turned to 270 degrees
- moved R31 110.2 mm to (196.2, 89.2), turned to 270 degrees
- moved D6 106.7 mm to (209.6, 87.0), turned to 180 degrees
- moved C15 105.1 mm to (201.9, 66.7)
- moved H3 96.1 mm to (311.8, 99.7), turned to 270 degrees
- moved U5 94.0 mm to (204.5, 98.4), turned to 270 degrees
- moved C14 91.5 mm to (201.3, 76.2), turned to 270 degrees
- moved L1 88.7 mm to (212.7, 76.8), turned to 90 degrees
- moved TP1 88.4 mm to (217.8, 87.6), turned to 270 degrees
- moved TP4 84.5 mm to (228.0, 101.6), turned to 270 degrees
- moved TP3 79.3 mm to (193.0, 62.9), turned to 270 degrees
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Connections:
- J5 pad 1: GND -> /H-
- J5 pad 2: /H- -> GND
Routing:
- net GND: track 27.4 -> 82.4 mm, vias 31 -> 27
- net +3V3: track 228.5 -> 174.7 mm, vias 4 -> 2
- net /SDDet: track 44.2 -> 0.00 mm, vias 1 -> 0
- net /SCK: track 41.1 -> 0.00 mm, vias 1 -> 0
- net /MISO: track 44.1 -> 3.18 mm, vias 1 -> 0
- net /MOSI: track 40.3 -> 0.00 mm, vias 1 -> 0
- net +5V: track 0.37 -> 40.6 mm
- net VCC: track 9.53 -> 42.9 mm
- net /SS: track 32.5 -> 0.00 mm, vias 1 -> 0
- net /RESET: track 24.2 -> 0.00 mm
- net Net-(R31-Pad1): track 0.00 -> 15.6 mm
- net Net-(D6-Pad1): track 0.00 -> 14.0 mm
- net /TOUT: track 139.7 -> 126.3 mm, vias 2 -> 0
- net /TempCtrl: track 121.8 -> 108.9 mm, vias 2 -> 0
- net Net-(C4-Pad1): track 13.1 -> 20.0 mm
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- removed copper zone on B.Cu, net GND
Other:
- board size 184.2 x 57.8 mm -> 266.1 x 97.2 mm
