File: ECAD/Heater.sch (KiCad schematic (older format))
At the start: 2 parts, among them J1 Conn_01x01_Female, J2 Conn_01x01_Female

Commit message: Cleanup
Renamed files, removed temp files
Connections:
- net +: no longer names the net of J1.1 (Pin_1), J2.1 (Pin_1)
Changed lines of the file:
@@
 $Descr A4 11693 8268
 encoding utf-8
-Sheet 2 2
+Sheet 1 1
 Title "PCB Heating Element"
 Date "2021-08-25"
@@
 Wire Wire Line
 	3150 1850 3800 1850
-Text HLabel 3050 1600 0    50   Input ~ 0
-+
-Text HLabel 3150 1600 2    50   Input ~ 0
--
 $Comp
 L Connector:Conn_01x01_Female J2
